Commit message: Update ur10_gripper.urdf

File: isaacgym/ur10_urdf/ur10_gripper.urdf (robot description, URDF)
Before this commit: robot ur10, 13 links, 12 joints
Links:
- added link ur10_leftfinger_tip; collision box size=0.013 0.004 0.0
- added link ur10_rightfinger_tip; collision box size=0.013 0.004 0.0
- added link ur_grip_site; visual sphere radius=0.005
Joints:
- added joint ur10_grip_vis_joint: type fixed, parent ee_link, child ur_grip_site, origin xyz=0 0 0.1625 rpy=0 0 0
- added joint ur10_leftfinger_tip_joint: type fixed, parent l_finger_link, child ur10_leftfinger_tip, origin xyz=0.035 -0.01 -0.015 rpy=0 0 0
- added joint ur10_rightfinger_tip_joint: type fixed, parent r_finger_link, child ur10_rightfinger_tip, origin xyz=0.035 0.01 -0.015 rpy=0 0 0
- joint l_finger_2_joint: origin xyz=0.049 0.026 0.000 rpy=0 0 0 -> xyz=0.049 0.026 0.0 rpy=0 0 0
- joint r_finger_2_joint: origin xyz=0.049 -0.026 0.000 rpy=0 0 0 -> xyz=0.049 -0.026 0.0 rpy=0 0 0
